File: Thermostat_Layout/schematic.sch (EAGLE design)
At the start: 11 parts, among them Q1 10 MHz, U1 ATMEGA328P-AU, U2 DS3231M+

Commit message: More schematic updates
Parts:
- added C3: (no value), rcl:C-EUC0402
- added RF24_CONN: (no value), jumper:JP4Q
- S1: device switch-omron:40-XX -> switch-omron:10-XX
Connections:
- net N$3 renamed UP_TEMP_BTN
- net N$4 renamed DWN_TEMP_BTN
- net N$5 renamed MODE_BTN
- net N$6 renamed FAN_BTN
- net N$7 renamed SETTINGS_BTN
- new net ANA_TEMP: U1.ADC6
- new net COOL_ON: U$1.GPB1
- new net FAN_ON: U$1.GPB2
- new net HEAT_ON: U$1.GPB0
- new net LCD_LED: U$1.GPB3
- new net REMOTE_BTN: U$1.GPA5
- new net RF_CE: RF24_CONN.3, U1.PC2
- new net RF_CS: RF24_CONN.4, U1.PC3
- new net SCHED_BTN: U$1.GPA6
- net +3V3: now also C3.1, RF24_CONN.2, U1.AREF
- net EXP_CS: now also U1.PC0
- net EXP_RST: now also U1.PC1
- net GND: now also C3.2, RF24_CONN.1
- net MISO: now also RF24_CONN.7
- net MOSI: now also RF24_CONN.6
- net SCK: now also RF24_CONN.5

Commit message: More layout changes
Parts:
- added BTN_HEADER: (no value), adafruit:PINHD-1X8BIG
- added IC1: LM50, linear:LM50
- added LCD_HEADER: (no value), pinhead:PINHD-1X16
- added R4: 10k, resistor:R-US_R0402
- added U3: AT25DF021-SSH-B, Atmel_By_element14_Batch_1-00:AT25DF021-SSH-B
- Q1: device crystal:CRYSTALHC49UP -> crystal:FC-12M
Connections:
- new net LCD_CONT: LCD_HEADER.3
- new net N$3: LCD_HEADER.15, R4.1
- net +3V3: now also IC1.+VS, LCD_HEADER.2, R4.2, U3.VCC, U3.~HOLD, U3.~WP
- net ANA_TEMP: now also IC1.VO
- net DWN_TEMP_BTN: now also BTN_HEADER.2
- net FAN_BTN: now also BTN_HEADER.4
- net GND: now also BTN_HEADER.8, IC1.GND, LCD_HEADER.1, LCD_HEADER.5, U3.GND
- net LCD_D4: now also LCD_HEADER.11
- net LCD_D5: now also LCD_HEADER.12
- net LCD_D6: now also LCD_HEADER.13
- net LCD_D7: now also LCD_HEADER.14
- net LCD_EN: now also LCD_HEADER.6
- net LCD_LED: now also LCD_HEADER.16
- net LCD_RS: now also LCD_HEADER.4
- net MEM_CS: now also U3.~CS
- net MISO: now also U3.SO
- net MODE_BTN: now also BTN_HEADER.3
- net MOSI: now also U3.SI
- net REMOTE_BTN: now also BTN_HEADER.6
- net SCHED_BTN: now also BTN_HEADER.7
- net SCK: now also U3.SCK
- net SETTINGS_BTN: now also BTN_HEADER.5
- net UP_TEMP_BTN: now also BTN_HEADER.1
Other:
- moved on the sheet: RF24_CONN

Commit message: Update schematic
Parts:
- added FTDI_HEADER: (no value), adafruit:PINHD-1X6B
- added JP1: (no value), adafruit:PINHD-1X3
- added R5: 220k, resistor:R-US_R0402
- added R6: 100k, resistor:R-US_R0402
- added TM1: (no value), adafruit:TRIMPOTTC33X
- R4: value 10k -> 220
Connections:
- new net +9V: JP1.2, R5.2
- new net BATT_MON: R5.1, R6.2, U1.ADC7
- net +3V3: now also FTDI_HEADER.3, JP1.1, TM1.A
- net GND: now also FTDI_HEADER.1, JP1.3, R6.1, TM1.E
- net LCD_CONT: now also TM1.S
- net UC_RST: now also FTDI_HEADER.6
- net UC_RX: now also FTDI_HEADER.5
- net UC_TX: now also FTDI_HEADER.4
Changed lines of the file:
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@@
 <part name="+3V8" library="supply1" library_urn="urn:adsk.eagle:library:371" deviceset="+3V3" device=""/>
 <part name="GND10" library="supply1" library_urn="urn:adsk.eagle:library:371" deviceset="GND" device=""/>
-<part name="R4" library="resistor" library_urn="urn:adsk.eagle:library:348" deviceset="R-US_" device="R0402" package3d_urn="urn:adsk.eagle:package:26058/1" value="10k"/>
+<part name="R4" library="resistor" library_urn="urn:adsk.eagle:library:348" deviceset="R-US_" device="R0402" package3d_urn="urn:adsk.eagle:package:26058/1" value="220"/>
+<part name="TM1" library="adafruit" library_urn="urn:adsk.eagle:library:420" deviceset="TRIMPOT" device="TC33X" package3d_urn="urn:adsk.eagle:package:6240639/1"/>
+<part name="+3V9" library="supply1" library_urn="urn:adsk.eagle:library:371" deviceset="+3V3" device=""/>
+<part name="GND11" library="supply1" library_urn="urn:adsk.eagle:library:371" deviceset="GND" device=""/>
+<part name="JP1" library="adafruit" library_urn="urn:adsk.eagle:library:420" deviceset="PINHD-1X3" device="" package3d_urn="urn:adsk.eagle:package:6240710/1"/>
+<part name="+3V10" library="supply1" library_urn="urn:adsk.eagle:library:371" deviceset="+3V3" device=""/>
+<part name="SUPPLY1" library="supply2" library_urn="urn:adsk.eagle:library:372" deviceset="+9V" device=""/>
+<part name="GND12" library="supply1" library_urn="urn:adsk.eagle:library:371" deviceset="GND" device=""/>
+<part name="R5" library="resistor" library_urn="urn:adsk.eagle:library:348" deviceset="R-US_" device="R0402" package3d_urn="urn:adsk.eagle:package:26058/1" value="220k"/>
+<part name="R6" library="resistor" library_urn="urn:adsk.eagle:library:348" deviceset="R-US_" device="R0402" package3d_urn="urn:adsk.eagle:package:26058/1" value="100k"/>
+<part name="SUPPLY2" library="supply2" library_urn="urn:adsk.eagle:library:372" deviceset="+9V" device=""/>
+<part name="GND13" library="supply1" library_urn="urn:adsk.eagle:library:371" deviceset="GND" device=""/>
+<part name="FTDI_HEADER" library="adafruit" library_urn="urn:adsk.eagle:library:420" deviceset="PINHD-1X6" device="B" package3d_urn="urn:adsk.eagle:package:6240714/1"/>
+<part name="+3V11" library="supply1" library_urn="urn:adsk.eagle:library:371" deviceset="+3V3" device=""/>
+<part name="GND14" library="supply1" library_urn="urn:adsk.eagle:library:371" deviceset="GND" device=""/>
 </parts>
 <sheets>
@@
 <instance part="GND10" gate="1" x="149.86" y="35.56" rot="R180"/>
 <instance part="R4" gate="G$1" x="190.5" y="0" rot="R90"/>
+<instance part="TM1" gate="G$1" x="226.06" y="25.4" rot="R180"/>
+<instance part="+3V9" gate="G$1" x="226.06" y="38.1"/>
+<instance part="GND11" gate="1" x="226.06" y="15.24"/>
+<instance part="JP1" gate="A" x="-43.18" y="88.9" rot="MR0"/>
+<instance part="+3V10" gate="G$1" x="-30.48" y="99.06"/>
+<instance part="SUPPLY1" gate="G$1" x="-22.86" y="99.06"/>
+<instance part="GND12" gate="1" x="-33.02" y="83.82"/>
+<instance part="R5" gate="G$1" x="-17.78" y="68.58" rot="R90"/>
+<instance part="R6" gate="G$1" x="-17.78" y="58.42" rot="R90"/>
+<instance part="SUPPLY2" gate="G$1" x="-17.78" y="76.2"/>
+<instance part="GND13" gate="1" x="-17.78" y="50.8"/>
+<instance part="FTDI_HEADER" gate="A" x="25.4" y="25.4" rot="MR0"/>
+<instance part="+3V11" gate="G$1" x="45.72" y="35.56"/>
+<instance part="GND14" gate="1" x="38.1" y="35.56" rot="R180"/>
 </instances>
 <busses>
@@
 <junction x="149.86" y="30.48"/>
 </segment>
+<segment>
+<pinref part="TM1" gate="G$1" pin="E"/>
+<pinref part="GND11" gate="1" pin="GND"/>
+<wire x1="226.06" y1="20.32" x2="226.06" y2="17.78" width="0.1524" layer="91"/>
+</segment>
+<segment>
+<pinref part="JP1" gate="A" pin="3"/>
+<pinref part="GND12" gate="1" pin="GND"/>
+<wire x1="-40.64" y1="86.36" x2="-33.02" y2="86.36" width="0.1524" layer="91"/>
+</segment>
+<segment>
+<pinref part="R6" gate="G$1" pin="1"/>
+<pinref part="GND13" gate="1" pin="GND"/>
+</segment>
+<segment>
+<pinref part="FTDI_HEADER" gate="A" pin="1"/>
+<wire x1="27.94" y1="33.02" x2="38.1" y2="33.02" width="0.1524" layer="91"/>
+<pinref part="GND14" gate="1" pin="GND"/>
+</segment>
 </net>
 <net name="UC_RST" class="0">
@@
 <wire x1="96.52" y1="96.52" x2="109.22" y2="96.52" width="0.1524" layer="91"/>
 <label x="99.06" y="96.52" size="1.778" layer="95"/>
+</segment>
+<segment>
+<pinref part="FTDI_HEADER" gate="A" pin="6"/>
+<wire x1="27.94" y1="20.32" x2="45.72" y2="20.32" width="0.1524" layer="91"/>
+<label x="35.56" y="20.32" size="1.778" layer="95"/>
 </segment>
 </net>
@@
 <junction x="162.56" y="27.94"/>
 </segment>
+<segment>
+<pinref part="+3V9" gate="G$1" pin="+3V3"/>
+<pinref part="TM1" gate="G$1" pin="A"/>
+<wire x1="226.06" y1="35.56" x2="226.06" y2="30.48" width="0.1524" layer="91"/>
+</segment>
+<segment>
+<pinref part="+3V10" gate="G$1" pin="+3V3"/>
+<wire x1="-30.48" y1="96.52" x2="-30.48" y2="91.44" width="0.1524" layer="91"/>
+<wire x1="-30.48" y1="91.44" x2="-40.64" y2="91.44" width="0.1524" layer="91"/>
+<pinref part="JP1" gate="A" pin="1"/>
+</segment>
+<segment>
+<pinref part="FTDI_HEADER" gate="A" pin="3"/>
+<pinref part="+3V11" gate="G$1" pin="+3V3"/>
+<wire x1="27.94" y1="27.94" x2="45.72" y2="27.94" width="0.1524" layer="91"/>
+<wire x1="45.72" y1="27.94" x2="45.72" y2="33.02" width="0.1524" layer="91"/>
+</segment>
 </net>
 <net name="LCD_RS" class="0">
@@
 <label x="101.6" y="88.9" size="1.778" layer="95"/>
 </segment>
+<segment>
+<pinref part="FTDI_HEADER" gate="A" pin="4"/>
+<wire x1="27.94" y1="25.4" x2="45.72" y2="25.4" width="0.1524" layer="91"/>
+<label x="35.56" y="25.4" size="1.778" layer="95"/>
+</segment>
 </net>
 <net name="UC_RX" class="0">
@@
 <wire x1="96.52" y1="91.44" x2="109.22" y2="91.44" width="0.1524" layer="91"/>
 <label x="101.6" y="91.44" size="1.778" layer="95"/>
+</segment>
+<segment>
+<pinref part="FTDI_HEADER" gate="A" pin="5"/>
+<wire x1="27.94" y1="22.86" x2="45.72" y2="22.86" width="0.1524" layer="91"/>
+<label x="35.56" y="22.86" size="1.778" layer="95"/>
 </segment>
 </net>
@@
 <label x="152.4" y="25.4" size="1.778" layer="95"/>
 </segment>
+<segment>
+<pinref part="TM1" gate="G$1" pin="S"/>
+<wire x1="220.98" y1="25.4" x2="208.28" y2="25.4" width="0.1524" layer="91"/>
+<label x="208.28" y="25.4" size="1.778" layer="95"/>
+</segment>
 </net>
 <net name="N$3" class="0">
@@
 </segment>
 </net>
+<net name="+9V" class="0">
+<segment>
+<pinref part="JP1" gate="A" pin="2"/>
+<pinref part="SUPPLY1" gate="G$1" pin="+9V"/>
+<wire x1="-40.64" y1="88.9" x2="-22.86" y2="88.9" width="0.1524" layer="91"/>
+<wire x1="-22.86" y1="88.9" x2="-22.86" y2="96.52" width="0.1524" layer="91"/>
+</segment>
+<segment>
+<pinref part="R5" gate="G$1" pin="2"/>
+<pinref part="SUPPLY2" gate="G$1" pin="+9V"/>
+</segment>
+</net>
+<net name="BATT_MON" class="0">
+<segment>
+<pinref part="R5" gate="G$1" pin="1"/>
+<pinref part="R6" gate="G$1" pin="2"/>
+<wire x1="-17.78" y1="63.5" x2="0" y2="63.5" width="0.1524" layer="91"/>
+<junction x="-17.78" y="63.5"/>
+<label x="-10.16" y="63.5" size="1.778" layer="95"/>
+</segment>
+<segment>
+<pinref part="U1" gate="A" pin="ADC7"/>
+<wire x1="60.96" y1="99.06" x2="40.64" y2="99.06" width="0.1524" layer="91"/>
+<label x="40.64" y="99.06" size="1.778" layer="95"/>
+</segment>
+</net>
