File: Thermostat_Layout/schematic.sch (EAGLE design)
At the start: 31 parts, among them IC1 LM50, IC2 MCP23017SO, IC3 MCP23017SO, Q1 10 MHz, U1 ATMEGA328P-AU, U2 DS3231M+, U3 AT25DF021-SSH-B, U4 VO14642AT, U5 VO14642AT, U6 VO14642AT

Commit message: Clean up schematic and board
Parts:
- removed IC3: MCP23017SO, microchip:MCP23017SO
- removed JP2: (no value), adafruit:PINHD-1X3CB
- added R10, R11: 1k, resistor:R-US_R0402
- IC2: value MCP23017SO -> MCP23S17SO; device microchip:MCP23017SO -> microchip:MCP23S17SO
- renumbered JP1 to POWER_CON, U$2 to BATT
Connections:
- net DWN_TEMP_BTN renamed DWN_BTN
- net UP_TEMP_BTN renamed UP_BTN
- removed net EXP_INTA: IC2.INTA, U1.PD2
- new net EXP_INT: IC2.INTA
- new net N$10: R11.2, U1.PD1
- new net N$13: U1.PD3
- new net N$9: R10.2, U1.PD0
- net +3V3: now also U1.VCC_2; no longer IC3.A0, IC3.VDD, JP2.1
- net EXP_CS: now also IC2.!CS, U1.PC0; no longer U1.PD7
- net EXP_RST: now also U1.PC1; no longer U1.PD6
- net FAN_HOT: now also AC_HEADER.1; no longer AC_HEADER.3
- net GND: now also U1.GND_2; no longer IC3.A1, IC3.A2, IC3.VSS, JP2.3
- net HEAT_HOT: now also AC_HEADER.3; no longer AC_HEADER.1
- net LCD_D0: now also LCD_HEADER.7; no longer IC3.GPA0
- net LCD_D1: now also LCD_HEADER.8; no longer IC3.GPA1
- net LCD_D2: now also LCD_HEADER.9; no longer IC3.GPA2
- net LCD_D3: now also LCD_HEADER.10; no longer IC3.GPA3
- net LCD_D4: now also U1.PD7; no longer IC3.GPA4
- net LCD_D5: now also U1.PD6; no longer IC3.GPA5
- net LCD_D6: now also U1.PD5; no longer IC3.GPA6
- net LCD_D7: now also U1.PD4; no longer IC3.GPA7
- net LCD_EN: now also U1.PB0; no longer IC3.GPB1
- net LCD_LED: now also IC2.GPB3; no longer IC3.GPB2
- net LCD_RS: now also U1.PB1; no longer IC3.GPB0
- net MISO: now also IC2.SO
- net MOSI: now also IC2.SI
- net RF_CE: now also U1.PC2; no longer U1.PB0
- net RF_CS: now also U1.PC3; no longer U1.PB1
- net SCK: now also IC2.SCK
- net SCL: no longer IC2.SCL, IC3.SCL
- net SDA: no longer IC2.SDA, IC3.SDA
- net UC_RST: no longer U1.PC6
- net UC_RX: now also R10.1; no longer U1.PD0
- net UC_TX: now also R11.1; no longer U1.PD1
Other:
- moved on the sheet: R2, R3
