File: Thermostat_Remote/Radio.sch (KiCad schematic (older format))
At the start: 0 parts

Commit message: Update remote sensor layout
Parts:
- added C10: 1.5pF, Capacitor_SMD:C_0402_1005Metric, symbol Device:C
- added C4: 33nF, Capacitor_SMD:C_0402_1005Metric, symbol Device:C
- added C5, C7: 22pF, Capacitor_SMD:C_0402_1005Metric, symbol Device:C
- added C6: 2.2nF, Capacitor_SMD:C_0402_1005Metric, symbol Device:C
- added C8: 4.7pF, Capacitor_SMD:C_0402_1005Metric, symbol Device:C
- added C9: 15pF, Capacitor_SMD:C_0402_1005Metric, symbol Device:C
- added J3: Conn_Coaxial, Connector_Coaxial:U.FL_Molex_MCRF_73412-0110_Vertical, symbol Connector:Conn_Coaxial
- added L1: 12nH, Inductor_SMD:L_0402_1005Metric, symbol Device:L
- added L2: 2.3nH, Inductor_SMD:L_0402_1005Metric, symbol Device:L
- added L3: 7.9nH, Inductor_SMD:L_0402_1005Metric, symbol Device:L
- added R6: 22kΩ, Resistors:0402, symbol Device:R_US
- added R7: 1MΩ, Resistor_SMD:R_0402_1005Metric, symbol Device:R_US
- added U4: nRF24L01P, Package_DFN_QFN:QFN-20-1EP_4x4mm_P0.5mm_EP2.5x2.5mm, symbol RF:nRF24L01P
- added Y2: 16MHz, Crystal:Crystal_SMD_SeikoEpson_MC405-2Pin_9.6x4.1mm, symbol Device:Crystal
Connections:
- new net: C7.1, R7.1, U4.10 (XC1), Y2.2
- new net: C6.2, C8.2, L2.2, U4.11 (VDD_PA)
- new net: L1.2, L2.1, U4.12 (ANT1)
- new net: L1.1, L3.1, U4.13 (ANT2)
- new net: R6.1, U4.16 (IREF)
- new net: C4.1, U4.19 (DVDD)
- new net: C5.1, R7.2, U4.9 (XC2), Y2.1
- new net: C9.2, L3.2
- new net: C10.1, C9.1, J3.1 (In)
- new net 3.3V: U4.15 (VDD), U4.18 (VDD), U4.7 (VDD)
- new net GND: C10.2, C4.2, C5.2, C6.1, C7.2, C8.1, J3.2 (Ext), R6.2, U4.14 (VSS), U4.17 (VSS), U4.20 (VSS), U4.8 (VSS)
- new net MISO: U4.5 (MISO)
- new net MOSI: U4.4 (MOSI)
- new net RF_CE: U4.1 (CE)
- new net RF_CSN: U4.2 (CSN)
- new net SCK: U4.3 (SCK)
