File: RemoteSensor/Layout/USB.sch (KiCad schematic (older format))
At the start: 18 parts

Commit message: Update sensor schematic
Parts:
- removed U?: FT230XS, Package_SO:SSOP-16_3.9x4.9mm_P0.635mm, symbol Interface_USB:FT230XS
- Q? (x2): symbol dk_Transistors-Bipolar-BJT-Single:MMBT2222A-TP -> RemoteSensor-rescue:MMBT2222A-TP-dk_Transistors-Bipolar-BJT-Single
Changed lines of the file:
@@
 EESchema Schematic File Version 4
-LIBS:RemoteSensor-cache
-EELAYER 29 0
+EELAYER 30 0
 EELAYER END
 $Descr A4 11693 8268
@@
 $EndDescr
 $Comp
-L Interface_USB:FT230XS U?
-U 1 1 5EF07365
-P 2150 2250
-F 0 "U?" H 2150 3131 50  0000 C CNN
-F 1 "FT230XS" H 2150 3040 50  0000 C CNN
-F 2 "Package_SO:SSOP-16_3.9x4.9mm_P0.635mm" H 2600 1600 50  0001 C CNN
-F 3 "http://www.ftdichip.com/Products/ICs/FT230X.html" H 2150 2250 50  0001 C CNN
-	1    2150 2250
-	1    0    0    -1
-$EndComp
-$Comp
 L Device:Ferrite_Bead FB?
 U 1 1 5EF07BAD
@@
 L Jumper:Jumper_2_Open JP?
 U 1 1 5EF0D6FF
-P 7200 3500
-F 0 "JP?" H 7200 3735 50  0000 C CNN
-F 1 "Jumper_2_Open" H 7200 3644 50  0000 C CNN
-F 2 "Jumper:SolderJumper-2_P1.3mm_Open_Pad1.0x1.5mm" H 7200 3500 50  0001 C CNN
-F 3 "~" H 7200 3500 50  0001 C CNN
-	1    7200 3500
+P 7200 3600
+F 0 "JP?" H 7200 3835 50  0000 C CNN
+F 1 "Jumper_2_Open" H 7200 3744 50  0000 C CNN
+F 2 "Jumper:SolderJumper-2_P1.3mm_Open_Pad1.0x1.5mm" H 7200 3600 50  0001 C CNN
+F 3 "~" H 7200 3600 50  0001 C CNN
+	1    7200 3600
 	1    0    0    -1
 $EndComp
@@
 	7650 3400 6600 3400
 Wire Wire Line
-	6600 3500 7000 3500
-$Comp
-L SparkFun-PowerSymbols:V_USB #SUPPLY?
+	6600 3600 7000 3600
+$Comp
+L RemoteSensor-rescue:V_USB-SparkFun-PowerSymbols #SUPPLY?
 U 1 1 5EF0F32D
 P 5800 2200
@@
 PRG_TX
 $Comp
-L dk_Transistors-Bipolar-BJT-Single:MMBT2222A-TP Q?
+L RemoteSensor-rescue:MMBT2222A-TP-dk_Transistors-Bipolar-BJT-Single Q?
 U 1 1 5EF2CE7F
 P 2600 5500
@@
 $EndComp
 $Comp
-L dk_Transistors-Bipolar-BJT-Single:MMBT2222A-TP Q?
+L RemoteSensor-rescue:MMBT2222A-TP-dk_Transistors-Bipolar-BJT-Single Q?
 U 1 1 5EF2EBF2
 P 2600 6350
@@
 RST
 Wire Wire Line
-	7400 3500 8600 3500
+	7400 3600 8600 3600
 Wire Wire Line
 	8050 3400 8600 3400
@@
 	5800 4850 6000 4850
 $Comp
-L SparkFun-PowerSymbols:GND #GND?
+L RemoteSensor-rescue:GND-SparkFun-PowerSymbols #GND?
 U 1 1 5EF4CBA7
 P 6000 4850
@@
 $EndComp
 Connection ~ 6000 4850
+Text Label 8600 3600 2    50   ~ 0
+DTR
 $EndSCHEMATC

Commit message: Add footprints and component values
Parts:
- C10, C8, C9: renamed from C?; footprint (none) -> Capacitor_SMD:C_0603_1608Metric_Pad1.05x0.95mm_HandSolder
- D3, D4: renamed from D?; footprint (none) -> LED_SMD:LED_0603_1608Metric_Pad1.05x0.95mm_HandSolder
- FB1: renamed from FB?; footprint (none) -> Resistor_SMD:R_0603_1608Metric_Pad1.05x0.95mm_HandSolder
- R23, R24: renamed from R?; value R_US -> 10k; footprint (none) -> Resistor_SMD:R_0603_1608Metric_Pad1.05x0.95mm_HandSolder
- R25, R26: renamed from R?; footprint (none) -> Resistor_SMD:R_0603_1608Metric_Pad1.05x0.95mm_HandSolder
- R27, R28: renamed from R?; value R_US -> 100; footprint (none) -> Resistor_SMD:R_0603_1608Metric_Pad1.05x0.95mm_HandSolder
- gave numbers to parts that had none: 5
Changed lines of the file:
@@
 $EndDescr
 $Comp
-L Device:Ferrite_Bead FB?
+L Device:Ferrite_Bead FB1
 U 1 1 5EF07BAD
 P 5800 2350
-F 0 "FB?" H 5663 2304 50  0000 R CNN
+F 0 "FB1" H 5663 2304 50  0000 R CNN
 F 1 "Ferrite_Bead" H 5663 2395 50  0000 R CNN
-F 2 "" V 5730 2350 50  0001 C CNN
+F 2 "Resistor_SMD:R_0603_1608Metric_Pad1.05x0.95mm_HandSolder" V 5730 2350 50  0001 C CNN
 F 3 "~" H 5800 2350 50  0001 C CNN
 	1    5800 2350
@@
 $EndComp
 $Comp
-L Device:R_US R?
+L Device:R_US R25
 U 1 1 5EF0826F
 P 4400 3500
-F 0 "R?" V 4195 3500 50  0000 C CNN
+F 0 "R25" V 4195 3500 50  0000 C CNN
 F 1 "27" V 4286 3500 50  0000 C CNN
-F 2 "" V 4440 3490 50  0001 C CNN
+F 2 "Resistor_SMD:R_0603_1608Metric_Pad1.05x0.95mm_HandSolder" V 4440 3490 50  0001 C CNN
 F 3 "~" H 4400 3500 50  0001 C CNN
 	1    4400 3500
@@
 $EndComp
 $Comp
-L Device:R_US R?
+L Device:R_US R26
 U 1 1 5EF088E2
 P 4800 3600
-F 0 "R?" V 4595 3600 50  0000 C CNN
+F 0 "R26" V 4595 3600 50  0000 C CNN
 F 1 "27" V 4686 3600 50  0000 C CNN
-F 2 "" V 4840 3590 50  0001 C CNN
+F 2 "Resistor_SMD:R_0603_1608Metric_Pad1.05x0.95mm_HandSolder" V 4840 3590 50  0001 C CNN
 F 3 "~" H 4800 3600 50  0001 C CNN
 	1    4800 3600
@@
 	5050 3800 5200 3800
 $Comp
-L Device:C C?
+L Device:C C10
 U 1 1 5EF0B19A
 P 5050 4150
-F 0 "C?" H 5165 4196 50  0000 L CNN
+F 0 "C10" H 5165 4196 50  0000 L CNN
 F 1 "100n" H 5165 4105 50  0000 L CNN
-F 2 "" H 5088 4000 50  0001 C CNN
+F 2 "Capacitor_SMD:C_0603_1608Metric_Pad1.05x0.95mm_HandSolder" H 5088 4000 50  0001 C CNN
 F 3 "~" H 5050 4150 50  0001 C CNN
 	1    5050 4150
@@
 Connection ~ 5050 3200
 $Comp
-L Jumper:Jumper_2_Open JP?
+L Jumper:Jumper_2_Open JP1
 U 1 1 5EF0D6FF
 P 7200 3600
-F 0 "JP?" H 7200 3835 50  0000 C CNN
+F 0 "JP1" H 7200 3835 50  0000 C CNN
 F 1 "Jumper_2_Open" H 7200 3744 50  0000 C CNN
 F 2 "Jumper:SolderJumper-2_P1.3mm_Open_Pad1.0x1.5mm" H 7200 3600 50  0001 C CNN
@@
 $EndComp
 $Comp
-L Jumper:Jumper_2_Open JP?
+L Jumper:Jumper_2_Open JP2
 U 1 1 5EF0E1DD
 P 7850 3400
-F 0 "JP?" H 7850 3635 50  0000 C CNN
+F 0 "JP2" H 7850 3635 50  0000 C CNN
 F 1 "Jumper_2_Open" H 7850 3544 50  0000 C CNN
 F 2 "Jumper:SolderJumper-2_P1.3mm_Open_Pad1.0x1.5mm" H 7850 3400 50  0001 C CNN
@@
 	6600 3600 7000 3600
 $Comp
-L RemoteSensor-rescue:V_USB-SparkFun-PowerSymbols #SUPPLY?
+L RemoteSensor-rescue:V_USB-SparkFun-PowerSymbols #SUPPLY0122
 U 1 1 5EF0F32D
 P 5800 2200
-F 0 "#SUPPLY?" H 5850 2200 45  0001 L BNN
+F 0 "#SUPPLY0122" H 5850 2200 45  0001 L BNN
 F 1 "V_USB" H 5800 2476 45  0000 C CNN
 F 2 "XXX-00000" H 5800 2381 60  0000 C CNN
@@
 $EndComp
 $Comp
-L Device:LED D?
+L Device:LED D3
 U 1 1 5EF0F904
 P 6750 4800
-F 0 "D?" V 6697 4878 50  0000 L CNN
+F 0 "D3" V 6697 4878 50  0000 L CNN
 F 1 "LED" V 6788 4878 50  0000 L CNN
-F 2 "" H 6750 4800 50  0001 C CNN
+F 2 "LED_SMD:LED_0603_1608Metric_Pad1.05x0.95mm_HandSolder" H 6750 4800 50  0001 C CNN
 F 3 "~" H 6750 4800 50  0001 C CNN
 	1    6750 4800
@@
 $EndComp
 $Comp
-L Device:LED D?
+L Device:LED D4
 U 1 1 5EF109F5
 P 7150 4800
-F 0 "D?" V 7097 4878 50  0000 L CNN
+F 0 "D4" V 7097 4878 50  0000 L CNN
 F 1 "LED" V 7188 4878 50  0000 L CNN
-F 2 "" H 7150 4800 50  0001 C CNN
+F 2 "LED_SMD:LED_0603_1608Metric_Pad1.05x0.95mm_HandSolder" H 7150 4800 50  0001 C CNN
 F 3 "~" H 7150 4800 50  0001 C CNN
 	1    7150 4800
@@
 	7150 4200 7150 4650
 $Comp
-L Device:R_US R?
+L Device:R_US R27
 U 1 1 5EF1163C
 P 6750 5100
-F 0 "R?" H 6818 5146 50  0000 L CNN
-F 1 "R_US" H 6818 5055 50  0000 L CNN
-F 2 "" V 6790 5090 50  0001 C CNN
+F 0 "R27" H 6818 5146 50  0000 L CNN
+F 1 "100" H 6818 5055 50  0000 L CNN
+F 2 "Resistor_SMD:R_0603_1608Metric_Pad1.05x0.95mm_HandSolder" V 6790 5090 50  0001 C CNN
 F 3 "~" H 6750 5100 50  0001 C CNN
 	1    6750 5100
@@
 $EndComp
 $Comp
-L Device:R_US R?
+L Device:R_US R28
 U 1 1 5EF11D39
 P 7150 5100
-F 0 "R?" H 7218 5146 50  0000 L CNN
-F 1 "R_US" H 7218 5055 50  0000 L CNN
-F 2 "" V 7190 5090 50  0001 C CNN
+F 0 "R28" H 7218 5146 50  0000 L CNN
+F 1 "100" H 7218 5055 50  0000 L CNN
+F 2 "Resistor_SMD:R_0603_1608Metric_Pad1.05x0.95mm_HandSolder" V 7190 5090 50  0001 C CNN
 F 3 "~" H 7150 5100 50  0001 C CNN
 	1    7150 5100
@@
 VCCIO
 $Comp
-L Device:C C?
+L Device:C C9
 U 1 1 5EF16A27
 P 4650 4150
-F 0 "C?" H 4765 4196 50  0000 L CNN
+F 0 "C9" H 4765 4196 50  0000 L CNN
 F 1 "47p" H 4765 4105 50  0000 L CNN
-F 2 "" H 4688 4000 50  0001 C CNN
+F 2 "Capacitor_SMD:C_0603_1608Metric_Pad1.05x0.95mm_HandSolder" H 4688 4000 50  0001 C CNN
 F 3 "~" H 4650 4150 50  0001 C CNN
 	1    4650 4150
@@
 $EndComp
 $Comp
-L Device:C C?
+L Device:C C8
 U 1 1 5EF171E4
 P 4250 4150
-F 0 "C?" H 4365 4196 50  0000 L CNN
+F 0 "C8" H 4365 4196 50  0000 L CNN
 F 1 "47p" H 4365 4105 50  0000 L CNN
-F 2 "" H 4288 4000 50  0001 C CNN
+F 2 "Capacitor_SMD:C_0603_1608Metric_Pad1.05x0.95mm_HandSolder" H 4288 4000 50  0001 C CNN
 F 3 "~" H 4250 4150 50  0001 C CNN
 	1    4250 4150
@@
 PRG_TX
 $Comp
-L RemoteSensor-rescue:MMBT2222A-TP-dk_Transistors-Bipolar-BJT-Single Q?
+L RemoteSensor-rescue:MMBT2222A-TP-dk_Transistors-Bipolar-BJT-Single Q4
 U 1 1 5EF2CE7F
 P 2600 5500
-F 0 "Q?" H 2788 5553 60  0000 L CNN
+F 0 "Q4" H 2788 5553 60  0000 L CNN
 F 1 "MMBT2222A-TP" H 2788 5447 60  0000 L CNN
 F 2 "digikey-footprints:SOT-23-3" H 2800 5700 60  0001 L CNN
@@
 $EndComp
 $Comp
-L RemoteSensor-rescue:MMBT2222A-TP-dk_Transistors-Bipolar-BJT-Single Q?
+L RemoteSensor-rescue:MMBT2222A-TP-dk_Transistors-Bipolar-BJT-Single Q5
 U 1 1 5EF2EBF2
 P 2600 6350
-F 0 "Q?" H 2788 6297 60  0000 L CNN
+F 0 "Q5" H 2788 6297 60  0000 L CNN
 F 1 "MMBT2222A-TP" H 2788 6403 60  0000 L CNN
 F 2 "digikey-footprints:SOT-23-3" H 2800 6550 60  0001 L CNN
@@
 $EndComp
 $Comp
-L Device:R_US R?
+L Device:R_US R23
 U 1 1 5EF30FEC
 P 2150 5500
-F 0 "R?" V 1945 5500 50  0000 C CNN
-F 1 "R_US" V 2036 5500 50  0000 C CNN
-F 2 "" V 2190 5490 50  0001 C CNN
+F 0 "R23" V 1945 5500 50  0000 C CNN
+F 1 "10k" V 2036 5500 50  0000 C CNN
+F 2 "Resistor_SMD:R_0603_1608Metric_Pad1.05x0.95mm_HandSolder" V 2190 5490 50  0001 C CNN
 F 3 "~" H 2150 5500 50  0001 C CNN
 	1    2150 5500
@@
 $EndComp
 $Comp
-L Device:R_US R?
+L Device:R_US R24
 U 1 1 5EF32BAD
 P 2150 6350
-F 0 "R?" V 2250 6350 50  0000 C CNN
-F 1 "R_US" V 2350 6350 50  0000 C CNN
-F 2 "" V 2190 6340 50  0001 C CNN
+F 0 "R24" V 2250 6350 50  0000 C CNN
+F 1 "10k" V 2350 6350 50  0000 C CNN
+F 2 "Resistor_SMD:R_0603_1608Metric_Pad1.05x0.95mm_HandSolder" V 2190 6340 50  0001 C CNN
 F 3 "~" H 2150 6350 50  0001 C CNN
 	1    2150 6350
@@
 RTS
 $Comp
-L Interface_USB:FT231XS U?
+L Interface_USB:FT231XS U10
 U 1 1 5EF43B07
 P 5900 3800
-F 0 "U?" H 5900 4881 50  0000 C CNN
+F 0 "U10" H 5900 4881 50  0000 C CNN
 F 1 "FT231XS" H 5900 4790 50  0000 C CNN
 F 2 "Package_SO:SSOP-20_3.9x8.7mm_P0.635mm" H 6500 2850 50  0001 C CNN
@@
 	5800 4850 6000 4850
 $Comp
-L RemoteSensor-rescue:GND-SparkFun-PowerSymbols #GND?
+L RemoteSensor-rescue:GND-SparkFun-PowerSymbols #GND0113
 U 1 1 5EF4CBA7
 P 6000 4850
-F 0 "#GND?" H 6050 4800 45  0001 L BNN
+F 0 "#GND0113" H 6050 4800 45  0001 L BNN
 F 1 "GND" H 6000 4680 45  0000 C CNN
 F 2 "" H 6000 4750 60  0001 C CNN

Commit message: Update PCB layout
Parts:
- removed D3, D4: LED, LED_SMD:LED_0603_1608Metric_Pad1.05x0.95mm_HandSolder, symbol Device:LED
- removed R27, R28: 100, Resistor_SMD:R_0603_1608Metric_Pad1.05x0.95mm_HandSolder, symbol Device:R_US
Connections:
- wire segments 52 -> 44
Changed lines of the file:
@@
 Connection ~ 5050 3800
-Wire Wire Line
-	4950 3600 5200 3600
 Wire Wire Line
 	4550 3500 5200 3500
@@
 	1    0    0    -1
 $EndComp
-$Comp
-L Device:LED D3
-U 1 1 5EF0F904
-P 6750 4800
-F 0 "D3" V 6697 4878 50  0000 L CNN
-F 1 "LED" V 6788 4878 50  0000 L CNN
-F 2 "LED_SMD:LED_0603_1608Metric_Pad1.05x0.95mm_HandSolder" H 6750 4800 50  0001 C CNN
-F 3 "~" H 6750 4800 50  0001 C CNN
-	1    6750 4800
-	0    1    1    0
-$EndComp
-$Comp
-L Device:LED D4
-U 1 1 5EF109F5
-P 7150 4800
-F 0 "D4" V 7097 4878 50  0000 L CNN
-F 1 "LED" V 7188 4878 50  0000 L CNN
-F 2 "LED_SMD:LED_0603_1608Metric_Pad1.05x0.95mm_HandSolder" H 7150 4800 50  0001 C CNN
-F 3 "~" H 7150 4800 50  0001 C CNN
-	1    7150 4800
-	0    1    1    0
-$EndComp
-Wire Wire Line
-	6600 4300 6750 4300
-Wire Wire Line
-	6750 4300 6750 4650
-Wire Wire Line
-	6600 4200 7150 4200
-Wire Wire Line
-	7150 4200 7150 4650
-$Comp
-L Device:R_US R27
-U 1 1 5EF1163C
-P 6750 5100
-F 0 "R27" H 6818 5146 50  0000 L CNN
-F 1 "100" H 6818 5055 50  0000 L CNN
-F 2 "Resistor_SMD:R_0603_1608Metric_Pad1.05x0.95mm_HandSolder" V 6790 5090 50  0001 C CNN
-F 3 "~" H 6750 5100 50  0001 C CNN
-	1    6750 5100
-	1    0    0    -1
-$EndComp
-$Comp
-L Device:R_US R28
-U 1 1 5EF11D39
-P 7150 5100
-F 0 "R28" H 7218 5146 50  0000 L CNN
-F 1 "100" H 7218 5055 50  0000 L CNN
-F 2 "Resistor_SMD:R_0603_1608Metric_Pad1.05x0.95mm_HandSolder" V 7190 5090 50  0001 C CNN
-F 3 "~" H 7150 5100 50  0001 C CNN
-	1    7150 5100
-	1    0    0    -1
-$EndComp
-Wire Wire Line
-	6750 5250 6750 5400
-Wire Wire Line
-	6750 5400 7150 5400
-Wire Wire Line
-	7150 5400 7150 5250
-Wire Wire Line
-	7150 5400 7900 5400
-Connection ~ 7150 5400
-Text Label 7900 5400 2    50   ~ 0
-VCCIO
 $Comp
 L Device:C C9
@@
 Text Label 8600 3400 2    50   ~ 0
 RTS
+Wire Wire Line
+	4650 4300 4650 4850
+Wire Wire Line
+	4650 4850 5800 4850
+Wire Wire Line
+	6000 4850 6000 4700
+Wire Wire Line
+	5800 4700 5800 4850
+Connection ~ 5800 4850
+Wire Wire Line
+	5800 4850 6000 4850
+$Comp
+L RemoteSensor-rescue:GND-SparkFun-PowerSymbols #GND0113
+U 1 1 5EF4CBA7
+P 6000 4850
+F 0 "#GND0113" H 6050 4800 45  0001 L BNN
+F 1 "GND" H 6000 4680 45  0000 C CNN
+F 2 "" H 6000 4750 60  0001 C CNN
+F 3 "" H 6000 4750 60  0001 C CNN
+	1    6000 4850
+	1    0    0    -1
+$EndComp
+Connection ~ 6000 4850
+Text Label 8600 3600 2    50   ~ 0
+DTR
+Wire Wire Line
+	4950 3600 5200 3600
 $Comp
 L Interface_USB:FT231XS U10
@@
 	1    0    0    -1
 $EndComp
-Wire Wire Line
-	4650 4300 4650 4850
-Wire Wire Line
-	4650 4850 5800 4850
-Wire Wire Line
-	6000 4850 6000 4700
-Wire Wire Line
-	5800 4700 5800 4850
-Connection ~ 5800 4850
-Wire Wire Line
-	5800 4850 6000 4850
-$Comp
-L RemoteSensor-rescue:GND-SparkFun-PowerSymbols #GND0113
-U 1 1 5EF4CBA7
-P 6000 4850
-F 0 "#GND0113" H 6050 4800 45  0001 L BNN
-F 1 "GND" H 6000 4680 45  0000 C CNN
-F 2 "" H 6000 4750 60  0001 C CNN
-F 3 "" H 6000 4750 60  0001 C CNN
-	1    6000 4850
-	1    0    0    -1
-$EndComp
-Connection ~ 6000 4850
-Text Label 8600 3600 2    50   ~ 0
-DTR
 $EndSCHEMATC

Commit message: Change what pins are used for i2c
Parts:
- C10, C8, C9: symbol Device:C -> RemoteSensor-rescue:C-Device
- FB1: symbol Device:Ferrite_Bead -> RemoteSensor-rescue:Ferrite_Bead-Device
- JP1, JP2: symbol Jumper:Jumper_2_Open -> RemoteSensor-rescue:Jumper_2_Open-Jumper
- R23, R24, R25, R26: symbol Device:R_US -> RemoteSensor-rescue:R_US-Device
- U10: symbol Interface_USB:FT231XS -> RemoteSensor-rescue:FT231XS-Interface_USB
Changed lines of the file:
@@
 $EndDescr
 $Comp
-L Device:Ferrite_Bead FB1
+L RemoteSensor-rescue:Ferrite_Bead-Device FB1
 U 1 1 5EF07BAD
 P 5800 2350
@@
 $EndComp
 $Comp
-L Device:R_US R25
+L RemoteSensor-rescue:R_US-Device R25
 U 1 1 5EF0826F
 P 4400 3500
@@
 $EndComp
 $Comp
-L Device:R_US R26
+L RemoteSensor-rescue:R_US-Device R26
 U 1 1 5EF088E2
 P 4800 3600
@@
 	5050 3800 5200 3800
 $Comp
-L Device:C C10
+L RemoteSensor-rescue:C-Device C10
 U 1 1 5EF0B19A
 P 5050 4150
@@
 Connection ~ 5050 3200
 $Comp
-L Jumper:Jumper_2_Open JP1
+L RemoteSensor-rescue:Jumper_2_Open-Jumper JP1
 U 1 1 5EF0D6FF
 P 7200 3600
@@
 $EndComp
 $Comp
-L Jumper:Jumper_2_Open JP2
+L RemoteSensor-rescue:Jumper_2_Open-Jumper JP2
 U 1 1 5EF0E1DD
 P 7850 3400
@@
 $EndComp
 $Comp
-L Device:C C9
+L RemoteSensor-rescue:C-Device C9
 U 1 1 5EF16A27
 P 4650 4150
@@
 $EndComp
 $Comp
-L Device:C C8
+L RemoteSensor-rescue:C-Device C8
 U 1 1 5EF171E4
 P 4250 4150
@@
 $EndComp
 $Comp
-L Device:R_US R23
+L RemoteSensor-rescue:R_US-Device R23
 U 1 1 5EF30FEC
 P 2150 5500
@@
 $EndComp
 $Comp
-L Device:R_US R24
+L RemoteSensor-rescue:R_US-Device R24
 U 1 1 5EF32BAD
 P 2150 6350
@@
 	4950 3600 5200 3600
 $Comp
-L Interface_USB:FT231XS U10
+L RemoteSensor-rescue:FT231XS-Interface_USB U10
 U 1 1 5EF43B07
 P 5900 3800

Commit message: Another layout
Parts:
- removed JP1, JP2: Jumper_2_Open, Jumper:SolderJumper-2_P1.3mm_Open_Pad1.0x1.5mm, symbol RemoteSensor-rescue:Jumper_2_Open-Jumper
- removed Q4, Q5: MMBT2222A-TP, digikey-footprints:SOT-23-3, symbol RemoteSensor-rescue:MMBT2222A-TP-dk_Transistors-Bipolar-BJT-Single
- removed R23, R24: 10k, Resistor_SMD:R_0603_1608Metric_Pad1.05x0.95mm_HandSolder, symbol RemoteSensor-rescue:R_US-Device
Changed lines of the file:
@@
 Connection ~ 5050 3200
-$Comp
-L RemoteSensor-rescue:Jumper_2_Open-Jumper JP1
-U 1 1 5EF0D6FF
-P 7200 3600
-F 0 "JP1" H 7200 3835 50  0000 C CNN
-F 1 "Jumper_2_Open" H 7200 3744 50  0000 C CNN
-F 2 "Jumper:SolderJumper-2_P1.3mm_Open_Pad1.0x1.5mm" H 7200 3600 50  0001 C CNN
-F 3 "~" H 7200 3600 50  0001 C CNN
-	1    7200 3600
-	1    0    0    -1
-$EndComp
-$Comp
-L RemoteSensor-rescue:Jumper_2_Open-Jumper JP2
-U 1 1 5EF0E1DD
-P 7850 3400
-F 0 "JP2" H 7850 3635 50  0000 C CNN
-F 1 "Jumper_2_Open" H 7850 3544 50  0000 C CNN
-F 2 "Jumper:SolderJumper-2_P1.3mm_Open_Pad1.0x1.5mm" H 7850 3400 50  0001 C CNN
-F 3 "~" H 7850 3400 50  0001 C CNN
-	1    7850 3400
-	1    0    0    -1
-$EndComp
-Wire Wire Line
-	7650 3400 6600 3400
-Wire Wire Line
-	6600 3600 7000 3600
 $Comp
 L RemoteSensor-rescue:V_USB-SparkFun-PowerSymbols #SUPPLY0122
@@
 PRG_TX
 Wire Wire Line
-	7400 3600 8600 3600
-Wire Wire Line
-	8050 3400 8600 3400
-Text Label 8600 3400 2    50   ~ 0
-RTS
-Wire Wire Line
 	4650 4300 4650 4850
 Wire Wire Line
@@
 $EndComp
 Connection ~ 6000 4850
-Text Label 8600 3600 2    50   ~ 0
-DTR
 Wire Wire Line
 	4950 3600 5200 3600
@@
 	1    0    0    -1
 $EndComp
-Text GLabel 3550 6750 2    50   Input ~ 0
-RST
-Text GLabel 3550 5100 2    50   Input ~ 0
-FLASH
-Text Label 1550 6350 0    50   ~ 0
-DTR
-Text Label 1550 5500 0    50   ~ 0
-RTS
-Wire Wire Line
-	2700 6750 3550 6750
-Wire Wire Line
-	2700 6550 2700 6750
-Wire Wire Line
-	2700 5100 3550 5100
-Wire Wire Line
-	2700 5300 2700 5100
-Wire Wire Line
-	2000 5500 1550 5500
-Wire Wire Line
-	2000 6350 1550 6350
-Wire Wire Line
-	2000 6200 2000 6350
-Wire Wire Line
-	2700 5850 2000 6200
-Wire Wire Line
-	2700 5700 2700 5850
-Wire Wire Line
-	2000 5650 2000 5500
-Wire Wire Line
-	2700 6050 2000 5650
-Wire Wire Line
-	2700 6150 2700 6050
-Wire Wire Line
-	2300 5500 2400 5500
-Wire Wire Line
-	2300 6350 2400 6350
-Connection ~ 2000 6350
-$Comp
-L RemoteSensor-rescue:R_US-Device R24
-U 1 1 5EF32BAD
-P 2150 6350
-F 0 "R24" V 2250 6350 50  0000 C CNN
-F 1 "10k" V 2350 6350 50  0000 C CNN
-F 2 "Resistor_SMD:R_0603_1608Metric_Pad1.05x0.95mm_HandSolder" V 2190 6340 50  0001 C CNN
-F 3 "~" H 2150 6350 50  0001 C CNN
-	1    2150 6350
-	0    1    1    0
-$EndComp
-Connection ~ 2000 5500
-$Comp
-L RemoteSensor-rescue:R_US-Device R23
-U 1 1 5EF30FEC
-P 2150 5500
-F 0 "R23" V 1945 5500 50  0000 C CNN
-F 1 "10k" V 2036 5500 50  0000 C CNN
-F 2 "Resistor_SMD:R_0603_1608Metric_Pad1.05x0.95mm_HandSolder" V 2190 5490 50  0001 C CNN
-F 3 "~" H 2150 5500 50  0001 C CNN
-	1    2150 5500
-	0    1    1    0
-$EndComp
-$Comp
-L RemoteSensor-rescue:MMBT2222A-TP-dk_Transistors-Bipolar-BJT-Single Q5
-U 1 1 5EF2EBF2
-P 2600 6350
-F 0 "Q5" H 2788 6297 60  0000 L CNN
-F 1 "MMBT2222A-TP" H 2788 6403 60  0000 L CNN
-F 2 "digikey-footprints:SOT-23-3" H 2800 6550 60  0001 L CNN
-F 3 "https://www.mccsemi.com/pdf/Products/MMBT2222A(SOT-23).pdf" H 2800 6650 60  0001 L CNN
-F 4 "MMBT2222ATPMSCT-ND" H 2800 6750 60  0001 L CNN "Digi-Key_PN"
-F 5 "MMBT2222A-TP" H 2800 6850 60  0001 L CNN "MPN"
-F 6 "Discrete Semiconductor Products" H 2800 6950 60  0001 L CNN "Category"
-F 7 "Transistors - Bipolar (BJT) - Single" H 2800 7050 60  0001 L CNN "Family"
-F 8 "https://www.mccsemi.com/pdf/Products/MMBT2222A(SOT-23).pdf" H 2800 7150 60  0001 L CNN "DK_Datasheet_Link"
-F 9 "/product-detail/en/micro-commercial-co/MMBT2222A-TP/MMBT2222ATPMSCT-ND/717394" H 2800 7250 60  0001 L CNN "DK_Detail_Page"
-F 10 "TRANS NPN 40V 0.6A SOT23" H 2800 7350 60  0001 L CNN "Description"
-F 11 "Micro Commercial Co" H 2800 7450 60  0001 L CNN "Manufacturer"
-F 12 "Active" H 2800 7550 60  0001 L CNN "Status"
-	1    2600 6350
-	1    0    0    1
-$EndComp
-$Comp
-L RemoteSensor-rescue:MMBT2222A-TP-dk_Transistors-Bipolar-BJT-Single Q4
-U 1 1 5EF2CE7F
-P 2600 5500
-F 0 "Q4" H 2788 5553 60  0000 L CNN
-F 1 "MMBT2222A-TP" H 2788 5447 60  0000 L CNN
-F 2 "digikey-footprints:SOT-23-3" H 2800 5700 60  0001 L CNN
-F 3 "https://www.mccsemi.com/pdf/Products/MMBT2222A(SOT-23).pdf" H 2800 5800 60  0001 L CNN
-F 4 "MMBT2222ATPMSCT-ND" H 2800 5900 60  0001 L CNN "Digi-Key_PN"
-F 5 "MMBT2222A-TP" H 2800 6000 60  0001 L CNN "MPN"
-F 6 "Discrete Semiconductor Products" H 2800 6100 60  0001 L CNN "Category"
-F 7 "Transistors - Bipolar (BJT) - Single" H 2800 6200 60  0001 L CNN "Family"
-F 8 "https://www.mccsemi.com/pdf/Products/MMBT2222A(SOT-23).pdf" H 2800 6300 60  0001 L CNN "DK_Datasheet_Link"
-F 9 "/product-detail/en/micro-commercial-co/MMBT2222A-TP/MMBT2222ATPMSCT-ND/717394" H 2800 6400 60  0001 L CNN "DK_Detail_Page"
-F 10 "TRANS NPN 40V 0.6A SOT23" H 2800 6500 60  0001 L CNN "Description"
-F 11 "Micro Commercial Co" H 2800 6600 60  0001 L CNN "Manufacturer"
-F 12 "Active" H 2800 6700 60  0001 L CNN "Status"
-	1    2600 5500
-	1    0    0    -1
-$EndComp
