File: RemoteSensor/Layout/Power.sch (KiCad schematic (older format))
At the start: 24 parts, among them J1 USB_B_Micro, J2 BATT_CONN, Q1 2N7002, U1 MCP73831-2-OT, U2 LD1117S33CTR, U3 BD48ExxG, U4 BD48ExxG, U5 LM3671MF

Commit message: Change how power is switched between battery and USB
Parts:
- removed C11, C3: 10u, Capacitor_SMD:C_0603_1608Metric_Pad1.05x0.95mm_HandSolder, symbol RemoteSensor-rescue:C-Device
- removed C4, C7: 4.7u, Capacitor_SMD:C_0603_1608Metric_Pad1.05x0.95mm_HandSolder, symbol RemoteSensor-rescue:C-Device
- removed C5: 1u, Capacitor_SMD:C_0603_1608Metric_Pad1.05x0.95mm_HandSolder, symbol RemoteSensor-rescue:C-Device
- removed C6: 0.1u, Capacitor_SMD:C_0603_1608Metric_Pad1.05x0.95mm_HandSolder, symbol RemoteSensor-rescue:C-Device
- removed D?: D, symbol Device:D
- removed Q1: 2N7002, digikey-footprints:SOT-23-3, symbol RemoteSensor-rescue:2N7002-dk_Transistors-FETs-MOSFETs-Single
- removed R5, R6: 10k, Resistor_SMD:R_0603_1608Metric_Pad1.05x0.95mm_HandSolder, symbol RemoteSensor-rescue:R_US-Device
- removed U2: LD1117S33CTR, digikey-footprints:SOT-223, symbol RemoteSensor-rescue:LD1117S33CTR-dk_PMIC-Voltage-Regulators-Linear
- added C11, C12, C13, C14, C15, C3, C4, C5, C6, C7: 47u, Capacitor_SMD:C_0603_1608Metric_Pad1.05x0.95mm_HandSolder, symbol Device:C
- added D3: D_Schottky, Diode_SMD:D_SOD-123, symbol Device:D_Schottky
- added Q1: Si3443DV, Si3443DV:Si3443DV, symbol Device:Q_PMOS_DGS
- added R5: 1, Resistor_SMD:R_0603_1608Metric_Pad1.05x0.95mm_HandSolder, symbol Device:R_US
Connections:
- net labels removed: FB, SW
- wire segments 84 -> 80
Other:
- moved on the sheet: J2, L1, R1, R2, R3, R4, U1, U3, U4, U5

Commit message: Another layout
Parts:
- added C16: 1u, Capacitor_SMD:C_0603_1608Metric_Pad1.05x0.95mm_HandSolder, symbol RemoteSensor-rescue:C-Device
- added C17: 0.1u, Capacitor_SMD:C_0603_1608Metric_Pad1.05x0.95mm_HandSolder, symbol RemoteSensor-rescue:C-Device
Connections:
- net GND: now also C16.2, C17.2
- net V_BATT: now also C16.1, C17.1
Changed lines of the file:
@@
 L RemoteSensor-rescue:GND-SparkFun-PowerSymbols #GND?
 U 1 1 5EEC211E
-P 7400 2300
+P 8200 2350
 AR Path="/5EEC211E" Ref="#GND?"  Part="1"
 AR Path="/5EE9FD3C/5EEC211E" Ref="#GND0104"  Part="1"
-F 0 "#GND0104" H 7450 2250 45  0001 L BNN
-F 1 "GND" H 7400 2130 45  0000 C CNN
-F 2 "" H 7400 2200 60  0001 C CNN
-F 3 "" H 7400 2200 60  0001 C CNN
-	1    7400 2300
+F 0 "#GND0104" H 8250 2300 45  0001 L BNN
+F 1 "GND" H 8200 2180 45  0000 C CNN
+F 2 "" H 8200 2250 60  0001 C CNN
+F 3 "" H 8200 2250 60  0001 C CNN
+	1    8200 2350
 	1    0    0    -1
 $EndComp
@@
 L RemoteSensor-rescue:V_BATT-SparkFun-PowerSymbols #SUPPLY?
 U 1 1 5EEC2137
-P 7400 1850
+P 8200 1850
 AR Path="/5EEC2137" Ref="#SUPPLY?"  Part="1"
 AR Path="/5EE9FD3C/5EEC2137" Ref="#SUPPLY0107"  Part="1"
-F 0 "#SUPPLY0107" H 7450 1850 45  0001 L BNN
-F 1 "V_BATT" H 7400 2126 45  0000 C CNN
-F 2 "XXX-00000" H 7400 2031 60  0000 C CNN
-F 3 "" H 7400 1850 60  0001 C CNN
-	1    7400 1850
-	1    0    0    -1
-$EndComp
-Wire Wire Line
-	7150 2050 7400 2050
-Wire Wire Line
-	7400 2050 7400 1850
+F 0 "#SUPPLY0107" H 8250 1850 45  0001 L BNN
+F 1 "V_BATT" H 8200 2126 45  0000 C CNN
+F 2 "XXX-00000" H 8200 2031 60  0000 C CNN
+F 3 "" H 8200 1850 60  0001 C CNN
+	1    8200 1850
+	1    0    0    -1
+$EndComp
 Wire Wire Line
 	7150 2150 7400 2150
-Wire Wire Line
-	7400 2150 7400 2300
 $Comp
 L RemoteSensor-rescue:L-Device L?
@@
 	1    0    0    -1
 $EndComp
+$Comp
+L RemoteSensor-rescue:C-Device C?
+U 1 1 5F6DE74C
+P 7800 2200
+AR Path="/5F6DE74C" Ref="C?"  Part="1"
+AR Path="/5EE9FD3C/5F6DE74C" Ref="C16"  Part="1"
+F 0 "C16" H 7915 2246 50  0000 L CNN
+F 1 "1u" H 7915 2155 50  0000 L CNN
+F 2 "Capacitor_SMD:C_0603_1608Metric_Pad1.05x0.95mm_HandSolder" H 7838 2050 50  0001 C CNN
+F 3 "~" H 7800 2200 50  0001 C CNN
+	1    7800 2200
+	1    0    0    -1
+$EndComp
+$Comp
+L RemoteSensor-rescue:C-Device C?
+U 1 1 5F6DF173
+P 8200 2200
+AR Path="/5F6DF173" Ref="C?"  Part="1"
+AR Path="/5EE9FD3C/5F6DF173" Ref="C17"  Part="1"
+F 0 "C17" H 8315 2246 50  0000 L CNN
+F 1 "0.1u" H 8315 2155 50  0000 L CNN
+F 2 "Capacitor_SMD:C_0603_1608Metric_Pad1.05x0.95mm_HandSolder" H 8238 2050 50  0001 C CNN
+F 3 "~" H 8200 2200 50  0001 C CNN
+	1    8200 2200
+	1    0    0    -1
+$EndComp
+Connection ~ 7800 2050
+Wire Wire Line
+	7800 2050 8200 2050
+Wire Wire Line
+	7150 2050 7800 2050
+Wire Wire Line
+	8200 1850 8200 2050
+Connection ~ 8200 2050
+Wire Wire Line
+	8200 2350 7800 2350
+Wire Wire Line
+	7400 2150 7400 2350
+Connection ~ 7800 2350
+Wire Wire Line
+	7800 2350 7400 2350
+Connection ~ 8200 2350
 $EndSCHEMATC

Commit message: Layout
Parts:
- L1: footprint Inductor_SMD:L_Taiyo-Yuden_NR-24xx_HandSoldering -> Inductor_SMD:L_Taiyo-Yuden_NR-30xx_HandSoldering
Changed lines of the file:
@@
 F 0 "L1" V 4190 4100 50  0000 C CNN
 F 1 "2.2u" V 4099 4100 50  0000 C CNN
-F 2 "Inductor_SMD:L_Taiyo-Yuden_NR-24xx_HandSoldering" H 4000 4100 50  0001 C CNN
+F 2 "Inductor_SMD:L_Taiyo-Yuden_NR-30xx_HandSoldering" H 4000 4100 50  0001 C CNN
 F 3 "~" H 4000 4100 50  0001 C CNN
 	1    4000 4100
